Commit message: replace flexiv headers and static lib files with latest branch in v2.xx develop

File: spec/flexiv_rizon4_kinematics.urdf (robot description, URDF)
Before this commit: robot A02L-MP, 9 links, 8 joints
Links:
- link base_link: geometry collision mesh filename=package://flexiv_description/meshes/A02L-M/collision/link0.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; visual mesh filename=package://flexiv_description/meshes/A02L-M/visual/link0.stl
- link link1: geometry collision mesh filename=package://flexiv_description/meshes/A02L-M/collision/link1.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; visual mesh filename=package://flexiv_description/meshes/A02L-M/visual/link1.stl
- link link2: geometry collision mesh filename=package://flexiv_description/meshes/A02L-M/collision/link2.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; visual mesh filename=package://flexiv_description/meshes/A02L-M/visual/link2.stl
- link link3: geometry collision mesh filename=package://flexiv_description/meshes/A02L-M/collision/link3.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; visual mesh filename=package://flexiv_description/meshes/A02L-M/visual/link3.stl
- link link4: geometry collision mesh filename=package://flexiv_description/meshes/A02L-M/collision/link4.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; visual mesh filename=package://flexiv_description/meshes/A02L-M/visual/link4.stl
- link link5: geometry collision mesh filename=package://flexiv_description/meshes/A02L-M/collision/link5.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; visual mesh filename=package://flexiv_description/meshes/A02L-M/visual/link5.stl
- link link6: geometry collision mesh filename=package://flexiv_description/meshes/A02L-M/collision/link6.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; visual mesh filename=package://flexiv_description/meshes/A02L-M/visual/link6.stl
- link link7: geometry collision mesh filename=package://flexiv_description/meshes/A02L-M/collision/link7.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; visual mesh filename=package://flexiv_description/meshes/A02L-M/visual/link7.stl
